Commit message: Start work on Reefscape Field world - Fix robot chassis being too short - Create new reefscape world
DOES NOT CONTAIN REQUIRED MODEL FILES. WILL NOT WORK FOR YOU.

More work on models

File: src/phyto_description/urdf/parts/swerve_chassis.xacro (robot description, xacro)
@@ -4,5 +4,5 @@
   <xacro:property name="chassis_length" value="0.661" />
   <xacro:property name="chassis_width" value="0.661" />
-  <xacro:property name="chassis_height" value="0.05588" />
+  <xacro:property name="chassis_height" value="0.059" />
   <xacro:property name="chassis_weight" value="19.0508795" />
     <xacro:macro name="square_chassis" params="prefix parent *origin">
